File: FinalBoardCircuits/BatteryCharger.kicad_sch (KiCad schematic)
At the start: 17 parts, among them IC4 BQ25302RTER, IC5 SI3483DDV-T1-BE3, J5 USB_B_Micro

Commit message: Added fuel guage
Added fuel guage circuit to the final design.
Parts:
- added IC1: LTC2941IMS8E#PBF, NaveenSymbols:SOP65P490X110-9N, symbol LTC2941IMS8E#PBF:LTC2941IMS8E#PBF
- added R1: 0.025, Resistor_SMD:R_0805_2012Metric_Pad1.20x1.40mm_HandSolder, symbol Device:R
Connections:
- net BAT_I-: now also IC1.1 (SENSE+), R1.1; no longer BT1.1 (+)
- new net FUEL_GUAGE-: BT1.1 (+), IC1.8 (SENSE-), R1.2
- new net GND: IC1.2 (GND)
- new net I2C1_SCL: IC1.3 (SCL)
- new net I2C1_SDA: IC1.6 (SDA)
- no-connect marks 2 -> 6
